Commit message: formatting and optimisation

File: inertials.urdf.xacro (robot description, xacro)
@@ -1,57 +1,64 @@
 <?xml version="1.0"?>
 <!--
-	Copyright (c) 2019 Andrey Stepanov (standmit)
-	Permission is hereby granted, free of charge, to any person obtaining a copy
-	of this software and associated documentation files (the "Software"), to deal
-	in the Software without restriction, including without limitation the rights
-	to use, copy, modify, merge, publish, distribute, sublicense, and/or sell
-	copies of the Software, and to permit persons to whom the Software is
-	furnished to do so, subject to the following conditions:
-	The above copyright notice and this permission notice shall be included in all
-	copies or substantial portions of the Software.
-	THE SOFTWARE IS PROVIDED "AS IS", WITHOUT WARRANTY OF ANY KIND, EXPRESS OR
-	IMPLIED, INCLUDING BUT NOT LIMITED TO THE WARRANTIES OF MERCHANTABILITY,
-	FITNESS FOR A PARTICULAR PURPOSE AND NONINFRINGEMENT. IN NO EVENT SHALL THE
-	AUTHORS OR COPYRIGHT HOLDERS BE LIABLE FOR ANY CLAIM, DAMAGES OR OTHER
-	LIABILITY, WHETHER IN AN ACTION OF CONTRACT, TORT OR OTHERWISE, ARISING FROM,
-	OUT OF OR IN CONNECTION WITH THE SOFTWARE OR THE USE OR OTHER DEALINGS IN THE
-	SOFTWARE.
+    Copyright (c) 2019 Andrey Stepanov (standmit)
+    Permission is hereby granted, free of charge, to any person obtaining a copy
+    of this software and associated documentation files (the "Software"), to deal
+    in the Software without restriction, including without limitation the rights
+    to use, copy, modify, merge, publish, distribute, sublicense, and/or sell
+    copies of the Software, and to permit persons to whom the Software is
+    furnished to do so, subject to the following conditions:
+    The above copyright notice and this permission notice shall be included in all
+    copies or substantial portions of the Software.
+    THE SOFTWARE IS PROVIDED "AS IS", WITHOUT WARRANTY OF ANY KIND, EXPRESS OR
+    IMPLIED, INCLUDING BUT NOT LIMITED TO THE WARRANTIES OF MERCHANTABILITY,
+    FITNESS FOR A PARTICULAR PURPOSE AND NONINFRINGEMENT. IN NO EVENT SHALL THE
+    AUTHORS OR COPYRIGHT HOLDERS BE LIABLE FOR ANY CLAIM, DAMAGES OR OTHER
+    LIABILITY, WHETHER IN AN ACTION OF CONTRACT, TORT OR OTHERWISE, ARISING FROM,
+    OUT OF OR IN CONNECTION WITH THE SOFTWARE OR THE USE OR OTHER DEALINGS IN THE
+    SOFTWARE.
 -->
 <robot xmlns:xacro="http://www.ros.org/wiki/xacro">
-	<xacro:macro name="cylinder_inertia" params="mass length radius">
-		<mass value="${mass}" />
-		<inertia
-			ixx="${mass*(3*radius*radius+length*length)/12}"
-			ixy="0"
-			ixz="0"
-			iyy="${mass*(3*radius*radius+length*length)/12}"
-			iyz="0"
-			izz="${mass*radius*radius/2}"
-		/>
-	</xacro:macro>
-	<xacro:macro name="box_inertia" params="mass size">
-	<xacro:property name="x" value="${size.split()[0]}" />
-	<xacro:property name="y" value="${size.split()[1]}" />
-	<xacro:property name="z" value="${size.split()[2]}" />
-		<mass value="${mass}" />
-		<inertia
-			ixx="${mass*(y*y+z*z)/12}"
-			ixy="0"
-			ixz="0"
-			iyy="${mass*(z*z+x*x)/12}"
-			iyz="0"
-			izz="${mass*(y*y+x*x)/12}"
-		/>
-	</xacro:macro>
-	<xacro:macro name="sphere_inertia" params="mass radius">
-		<mass value="${mass}" />
-		<inertia
-			ixx="${2*mass*radius*radius/5}"
-			ixy="0"
-			ixz="0"
-			iyy="${2*mass*radius*radius/5}"
-			iyz="0"
-			izz="${2*mass*radius*radius/5}"
-		/>
-	</xacro:macro>
+    <xacro:macro name="cylinder_inertia" params="mass length radius">
+        <xacro:property name="r_sq" value="${radius ** 2}" />
+        <xacro:property name="l_sq" value="${length ** 2}" />
+        <xacro:property name="horr_inertia" value="${mass * (3 * r_sq + l_sq) / 12}" />
+        <mass value="${mass}" />
+        <inertia
+            ixx="${horr_inertia}"
+            ixy="0"
+            ixz="0"
+            iyy="${horr_inertia}"
+            iyz="0"
+            izz="${mass * r_sq / 2}"
+        />
+    </xacro:macro>
+    <xacro:macro name="box_inertia" params="mass size">
+        <xacro:property name="x" value="${size.split()[0]}" />
+        <xacro:property name="y" value="${size.split()[1]}" />
+        <xacro:property name="z" value="${size.split()[2]}" />
+        <xacro:property name="x_sq" value="${x ** 2}" />
+        <xacro:property name="y_sq" value="${y ** 2}" />
+        <xacro:property name="z_sq" value="${z ** 2}" />
+        <mass value="${mass}" />
+        <inertia
+            ixx="${mass * (y_sq + z_sq) / 12}"
+            ixy="0"
+            ixz="0"
+            iyy="${mass * (z_sq + x_sq) / 12}"
+            iyz="0"
+            izz="${mass * (y_sq + x_sq) / 12}"
+        />
+    </xacro:macro>
+    <xacro:macro name="sphere_inertia" params="mass radius">
+        <xacro:property name="r_sq" value="${radius ** 2}" />
+        <mass value="${mass}" />
+        <inertia
+            ixx="${2 * mass * r_sq / 5}"
+            ixy="0"
+            ixz="0"
+            iyy="${2 * mass * r_sq / 5}"
+            iyz="0"
+            izz="${2 * mass * r_sq / 5}"
+        />
+    </xacro:macro>
 </robot>

File: simple_link.urdf.xacro (robot description, xacro)
@@ -1,20 +1,20 @@
 <?xml version="1.0"?>
 <!--
-	Copyright (c) 2019 Andrey Stepanov (standmit)
-	Permission is hereby granted, free of charge, to any person obtaining a copy
-	of this software and associated documentation files (the "Software"), to deal
-	in the Software without restriction, including without limitation the rights
-	to use, copy, modify, merge, publish, distribute, sublicense, and/or sell
-	copies of the Software, and to permit persons to whom the Software is
-	furnished to do so, subject to the following conditions:
-	The above copyright notice and this permission notice shall be included in all
-	copies or substantial portions of the Software.
-	THE SOFTWARE IS PROVIDED "AS IS", WITHOUT WARRANTY OF ANY KIND, EXPRESS OR
-	IMPLIED, INCLUDING BUT NOT LIMITED TO THE WARRANTIES OF MERCHANTABILITY,
-	FITNESS FOR A PARTICULAR PURPOSE AND NONINFRINGEMENT. IN NO EVENT SHALL THE
-	AUTHORS OR COPYRIGHT HOLDERS BE LIABLE FOR ANY CLAIM, DAMAGES OR OTHER
-	LIABILITY, WHETHER IN AN ACTION OF CONTRACT, TORT OR OTHERWISE, ARISING FROM,
-	OUT OF OR IN CONNECTION WITH THE SOFTWARE OR THE USE OR OTHER DEALINGS IN THE
-	SOFTWARE.
+    Copyright (c) 2019 Andrey Stepanov (standmit)
+    Permission is hereby granted, free of charge, to any person obtaining a copy
+    of this software and associated documentation files (the "Software"), to deal
+    in the Software without restriction, including without limitation the rights
+    to use, copy, modify, merge, publish, distribute, sublicense, and/or sell
+    copies of the Software, and to permit persons to whom the Software is
+    furnished to do so, subject to the following conditions:
+    The above copyright notice and this permission notice shall be included in all
+    copies or substantial portions of the Software.
+    THE SOFTWARE IS PROVIDED "AS IS", WITHOUT WARRANTY OF ANY KIND, EXPRESS OR
+    IMPLIED, INCLUDING BUT NOT LIMITED TO THE WARRANTIES OF MERCHANTABILITY,
+    FITNESS FOR A PARTICULAR PURPOSE AND NONINFRINGEMENT. IN NO EVENT SHALL THE
+    AUTHORS OR COPYRIGHT HOLDERS BE LIABLE FOR ANY CLAIM, DAMAGES OR OTHER
+    LIABILITY, WHETHER IN AN ACTION OF CONTRACT, TORT OR OTHERWISE, ARISING FROM,
+    OUT OF OR IN CONNECTION WITH THE SOFTWARE OR THE USE OR OTHER DEALINGS IN THE
+    SOFTWARE.
 -->
 <robot xmlns:xacro="http://www.ros.org/wiki/xacro">
